File: KiCad_Schematic_PCB/STM32.kicad_sch (KiCad schematic)
At the start: 9 parts, among them J208 Conn_02x07_Odd_Even, U201 STM32G0RBT6, Y201 16MHz

Commit message: Schematic_KiCad_v2
Parts:
- removed U201: STM32G0RBT6, Package_QFP:LQFP-64_10x10mm_P0.5mm, symbol STM32G0RBT6:STM32G0RBT6
- added C204: 100nF, Capacitor_SMD:C_0603_1608Metric_Pad1.08x0.95mm_HandSolder, symbol Device:C_Small
- added C205, C206: 10pF, Capacitor_SMD:C_0603_1608Metric_Pad1.08x0.95mm_HandSolder, symbol Device:C_Small
- added D201: GREEN, LED_SMD:LED_0603_1608Metric_Pad1.05x0.95mm_HandSolder, symbol Device:LED
- added D202: RED, LED_SMD:LED_0603_1608Metric_Pad1.05x0.95mm_HandSolder, symbol Device:LED
- added J209: JST_SUPP, Connector_JST:JST_XH_B6B-XH-A_1x06_P2.50mm_Vertical, symbol Connector_Generic:Conn_01x06
- added R202, R203: 1k, Resistor_SMD:R_0603_1608Metric_Pad0.98x0.95mm_HandSolder, symbol Device:R
- added U201: STM32G070RBT6, Package_QFP:LQFP-64_10x10mm_P0.5mm, symbol STM32G070RBT6:STM32G070RBT6
- C201, C202: value 10pF -> 100nF
- C203: value 100nF -> 4.7uF
Connections:
- net +3.3V: now also C201.1, C202.1, C203.1, U201.6 (VBat), U201.7 (VREF+), U201.8 (VDD)
- net CB1_OUT: now also U201.14 (PC1)
- net CB2_OUT: now also U201.15 (PC2)
- net GND: now also C204.2, C205.2, C206.2, R202.2, R203.2, U201.9 (VSS)
- net GPIO1_C1: now also U201.29 (PB2)
- net GPIO1_C2: now also U201.33 (PB13)
- net LED_CC: now also U201.23 (PA6)
- net NRST: now also C204.1, U201.12 (NRST); no longer C203.1
- net OE: now also U201.16 (PC3)
- net S0: now also U201.17 (PA0)
- net S1: now also U201.18 (PA1)
- net S2: now also U201.19 (PA2)
- net S3: now also U201.20 (PA3)
- net SCL_1: now also U201.37 (PA9)
- net SCL_2: now also U201.30 (PB10)
- net SDA_1: now also U201.42 (PA10)
- net SDA_2: now also U201.31 (PB11)
- net SYS_SWCLK: now also U201.46 (PA14)
- net SYS_SWDIO: now also U201.45 (PA13)
- net TIM_CC: now also U201.24 (PA7)
- net TIM_Driver1_CH1: now also U201.63 (PB9)
- net TIM_Driver1_CH1N: now also U201.61 (PB7)
- net TIM_Driver2_CH1: now also U201.62 (PB8)
- net TIM_Driver2_CH1N: now also U201.60 (PB6)
- net TIM_Encoder1_CH1: now also U201.48 (PC8)
- net TIM_Encoder1_CH2: now also U201.57 (PB3)
- net TIM_Encoder2_CH1: now also U201.58 (PB4)
- net TIM_Encoder2_CH2: now also U201.59 (PB5)
- net UART_STLink_RX: now also U201.26 (PC5)
- net UART_STLink_TX: now also U201.25 (PC4)
- net UART_XL320: now also U201.55 (PD5)
- net XSHUT_C1: now also U201.28 (PB1)
- net XSHUT_C2: now also U201.32 (PB12)
- net at R201.1: now also U201.11 (PF1_OSC_OUT)
- net at R201.2, Y201.1: now also C206.1; no longer C202.1
- net at Y201.3: now also C205.1, U201.10 (PF0_OSC_IN); no longer C201.1
- new net: D201.1 (K), R202.1
- new net: D202.1 (K), R203.1
- new net ADC: U201.27 (PB0)
- new net LED_GREEN: D201.2 (A), U201.1 (PC11)
- new net LED_RED: D202.2 (A), U201.2 (PC12)
- new net PC9: J209.1 (Pin_1), U201.49 (PC9)
- new net PD0: J209.2 (Pin_2), U201.50 (PD0)
- new net PD1: J209.3 (Pin_3), U201.51 (PD1)
- new net PD2: J209.4 (Pin_4), U201.52 (PD2)
- new net PD3: J209.5 (Pin_5), U201.53 (PD3)
- new net PD4: J209.6 (Pin_6), U201.54 (PD4)
- no-connect marks 35 -> 23
Other:
- note added: "LEDs"
- moved on the sheet: J208, JP201, JP202
