File: Hardware/KiCad_Schematic_PCB/Alimentation_v2.kicad_sch (KiCad schematic)
At the start: 12 parts

Commit message: Update Placement PCB
Parts:
- C501: value (none) -> 10uF; footprint (none) -> Capacitor_SMD:C_0603_1608Metric_Pad1.08x0.95mm_HandSolder
- C502: value (none) -> 22uF; footprint (none) -> Capacitor_SMD:C_0603_1608Metric_Pad1.08x0.95mm_HandSolder
- C503, C504: value (none) -> 1uF; footprint (none) -> Capacitor_SMD:C_0603_1608Metric_Pad1.08x0.95mm_HandSolder
- D501: value (none) -> LED; footprint (none) -> LED_SMD:LED_0603_1608Metric_Pad1.05x0.95mm_HandSolder
- J501: value (none) -> JST_switch; footprint (none) -> Connector_JST:JST_XH_B2B-XH-A_1x02_P2.50mm_Vertical
- R501: value (none) -> 1k; footprint (none) -> Resistor_SMD:R_0603_1608Metric_Pad0.98x0.95mm_HandSolder
- SW501: value (none) -> SW_SPDT; footprint (none) -> switch_robot:switch_pcb_robot
- U501: value (none) -> AZ1117-5.0; footprint (none) -> Package_TO_SOT_SMD:SOT-223-3_TabPin2
- U502: value (none) -> MCP1802x-xx02xOT; footprint (none) -> Package_TO_SOT_SMD:SOT-23-5
Changed lines of the file:
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@@
       (effects (font (size 1.27 1.27)) (justify right))
     )
-    (property "Value" "" (id 1) (at 228.854 139.7 0)
-      (effects (font (size 1.27 1.27)) (justify right))
-    )
-    (property "Footprint" "" (id 2) (at 223.52 139.7 0)
+    (property "Value" "1uF" (id 1) (at 228.854 139.7 0)
+      (effects (font (size 1.27 1.27)) (justify right))
+    )
+    (property "Footprint" "Capacitor_SMD:C_0603_1608Metric_Pad1.08x0.95mm_HandSolder" (id 2) (at 223.52 139.7 0)
       (effects (font (size 1.27 1.27)) hide)
     )
@@
     (in_bom yes) (on_board yes) (fields_autoplaced)
     (property "Reference" "U501" (id 0) (at 62.23 133.35 0))
-    (property "Value" "" (id 1) (at 62.23 135.89 0))
-    (property "Footprint" "" (id 2) (at 62.23 134.62 0)
+    (property "Value" "AZ1117-5.0" (id 1) (at 62.23 135.89 0))
+    (property "Footprint" "Package_TO_SOT_SMD:SOT-223-3_TabPin2" (id 2) (at 62.23 134.62 0)
       (effects (font (size 1.27 1.27) italic) hide)
     )
@@
     (in_bom yes) (on_board yes) (fields_autoplaced)
     (property "Reference" "J501" (id 0) (at 41.91 52.07 0))
-    (property "Value" "" (id 1) (at 41.91 54.61 0))
-    (property "Footprint" "" (id 2) (at 41.91 58.42 0)
+    (property "Value" "JST_switch" (id 1) (at 41.91 54.61 0))
+    (property "Footprint" "Connector_JST:JST_XH_B2B-XH-A_1x02_P2.50mm_Vertical" (id 2) (at 41.91 58.42 0)
       (effects (font (size 1.27 1.27)) hide)
     )
@@
       (effects (font (size 1.27 1.27)) (justify right))
     )
-    (property "Value" "" (id 1) (at 49.53 147.3135 0)
-      (effects (font (size 1.27 1.27)) (justify right))
-    )
-    (property "Footprint" "" (id 2) (at 52.07 146.05 0)
+    (property "Value" "10uF" (id 1) (at 49.53 147.3135 0)
+      (effects (font (size 1.27 1.27)) (justify right))
+    )
+    (property "Footprint" "Capacitor_SMD:C_0603_1608Metric_Pad1.08x0.95mm_HandSolder" (id 2) (at 52.07 146.05 0)
       (effects (font (size 1.27 1.27)) hide)
     )
@@
     (in_bom yes) (on_board yes)
     (property "Reference" "D501" (id 0) (at 166.37 54.9275 90))
-    (property "Value" "" (id 1) (at 166.37 57.4675 90))
-    (property "Footprint" "" (id 2) (at 160.02 54.61 0)
+    (property "Value" "LED" (id 1) (at 166.37 57.4675 90))
+    (property "Footprint" "LED_SMD:LED_0603_1608Metric_Pad1.05x0.95mm_HandSolder" (id 2) (at 160.02 54.61 0)
       (effects (font (size 1.27 1.27)) hide)
     )
@@
       (effects (font (size 1.27 1.27)) hide)
     )
-    (property "Value" "" (id 1) (at 46.99 135.763 0))
+    (property "Value" "+BATT" (id 1) (at 46.99 135.763 0))
     (property "Footprint" "" (id 2) (at 46.99 140.97 0)
       (effects (font (size 1.27 1.27)) hide)
@@
     (in_bom yes) (on_board yes)
     (property "Reference" "SW501" (id 0) (at 52.07 50.8 0))
-    (property "Value" "" (id 1) (at 54.61 53.34 0))
-    (property "Footprint" "" (id 2) (at 52.07 58.42 0)
+    (property "Value" "SW_SPDT" (id 1) (at 54.61 53.34 0))
+    (property "Footprint" "switch_robot:switch_pcb_robot" (id 2) (at 52.07 58.42 0)
       (effects (font (size 1.27 1.27)) hide)
     )
@@
       (effects (font (size 1.27 1.27)) hide)
     )
-    (property "Value" "" (id 1) (at 213.36 149.8599 0)
+    (property "Value" "GND" (id 1) (at 213.36 149.8599 0)
       (effects (font (size 1.27 1.27)) (justify right))
     )
@@
       (effects (font (size 1.27 1.27)) (justify right))
     )
-    (property "Value" "" (id 1) (at 193.04 138.9315 0)
-      (effects (font (size 1.27 1.27)) (justify right))
-    )
-    (property "Footprint" "" (id 2) (at 195.58 137.668 0)
+    (property "Value" "1uF" (id 1) (at 193.04 138.9315 0)
+      (effects (font (size 1.27 1.27)) (justify right))
+    )
+    (property "Footprint" "Capacitor_SMD:C_0603_1608Metric_Pad1.08x0.95mm_HandSolder" (id 2) (at 195.58 137.668 0)
       (effects (font (size 1.27 1.27)) hide)
     )
@@
       (effects (font (size 1.27 1.27)) hide)
     )
-    (property "Value" "" (id 1) (at 160.02 66.04 0))
+    (property "Value" "GND" (id 1) (at 160.02 66.04 0))
     (property "Footprint" "" (id 2) (at 160.02 60.96 0)
       (effects (font (size 1.27 1.27)) hide)
@@
       (effects (font (size 1.27 1.27)) hide)
     )
-    (property "Value" "" (id 1) (at 160.02 35.56 0))
+    (property "Value" "+3.3V" (id 1) (at 160.02 35.56 0))
     (property "Footprint" "" (id 2) (at 160.02 40.64 0)
       (effects (font (size 1.27 1.27)) hide)
@@
       (effects (font (size 1.27 1.27)) hide)
     )
-    (property "Value" "" (id 1) (at 228.6009 124.3782 0))
+    (property "Value" "+3.3V" (id 1) (at 228.6009 124.3782 0))
     (property "Footprint" "" (id 2) (at 228.6009 129.4582 0)
       (effects (font (size 1.27 1.27)) hide)
@@
       (effects (font (size 1.27 1.27)) (justify left))
     )
-    (property "Value" "" (id 1) (at 74.93 147.3262 0)
+    (property "Value" "22uF" (id 1) (at 74.93 147.3262 0)
       (effects (font (size 1.27 1.27)) (justify left))
     )
-    (property "Footprint" "" (id 2) (at 72.39 146.05 0)
+    (property "Footprint" "Capacitor_SMD:C_0603_1608Metric_Pad1.08x0.95mm_HandSolder" (id 2) (at 72.39 146.05 0)
       (effects (font (size 1.27 1.27)) hide)
     )
@@
       (effects (font (size 1.27 1.27)) hide)
     )
-    (property "Value" "" (id 1) (at 189.23 124.46 0))
+    (property "Value" "+5V" (id 1) (at 189.23 124.46 0))
     (property "Footprint" "" (id 2) (at 189.23 129.54 0)
       (effects (font (size 1.27 1.27)) hide)
@@
       (effects (font (size 1.27 1.27)) hide)
     )
-    (property "Value" "" (id 1) (at 64.77 157.4799 0)
+    (property "Value" "GND" (id 1) (at 64.77 157.4799 0)
       (effects (font (size 1.27 1.27)) (justify right))
     )
@@
     (in_bom yes) (on_board yes)
     (property "Reference" "R501" (id 0) (at 165.1 44.45 0))
-    (property "Value" "" (id 1) (at 165.1 46.99 0))
-    (property "Footprint" "" (id 2) (at 160.02 45.72 0)
+    (property "Value" "1k" (id 1) (at 165.1 46.99 0))
+    (property "Footprint" "Resistor_SMD:R_0603_1608Metric_Pad0.98x0.95mm_HandSolder" (id 2) (at 160.02 45.72 0)
       (effects (font (size 1.27 1.27)) hide)
     )
@@
       (effects (font (size 1.27 1.27)) hide)
     )
-    (property "Value" "" (id 1) (at 80.01 133.35 0))
+    (property "Value" "+5V" (id 1) (at 80.01 133.35 0))
     (property "Footprint" "" (id 2) (at 80.01 138.43 0)
       (effects (font (size 1.27 1.27)) hide)
@@
       (effects (font (size 1.27 1.27)) hide)
     )
-    (property "Value" "" (id 1) (at 60.96 46.99 0))
+    (property "Value" "+BATT" (id 1) (at 60.96 46.99 0))
     (property "Footprint" "" (id 2) (at 60.96 52.197 0)
       (effects (font (size 1.27 1.27)) hide)
@@
       (effects (font (size 1.27 1.27)) hide)
     )
-    (property "Value" "" (id 1) (at 49.53 72.3899 0)
+    (property "Value" "GND" (id 1) (at 49.53 72.3899 0)
       (effects (font (size 1.27 1.27)) (justify right))
     )
@@
     (in_bom yes) (on_board yes) (fields_autoplaced)
     (property "Reference" "U502" (id 0) (at 210.82 124.46 0))
-    (property "Value" "" (id 1) (at 210.82 127 0))
-    (property "Footprint" "" (id 2) (at 204.47 125.73 0)
+    (property "Value" "MCP1802x-xx02xOT" (id 1) (at 210.82 127 0))
+    (property "Footprint" "Package_TO_SOT_SMD:SOT-23-5" (id 2) (at 204.47 125.73 0)
       (effects (font (size 1.27 1.27) italic) (justify left) hide)
     )
