File: Hardware/KiCad_Schematic_PCB/capteurs_v2.kicad_sch (KiCad schematic)
At the start: 11 parts

Commit message: Update Placement PCB
Parts:
- J201: value (none) -> JST_Bordure_1; footprint (none) -> Connector_JST:JST_XH_B3B-XH-A_1x03_P2.50mm_Vertical
- J202: value (none) -> JST_TOF_1; footprint (none) -> Connector_JST:JST_XH_B6B-XH-A_1x06_P2.50mm_Vertical
- J203: value (none) -> JST_TOF_2; footprint (none) -> Connector_JST:JST_XH_B6B-XH-A_1x06_P2.50mm_Vertical
- J204: value (none) -> JST_Bordure_2; footprint (none) -> Connector_JST:JST_XH_B3B-XH-A_1x03_P2.50mm_Vertical
- J205: value (none) -> JST_Couleur_1A; footprint (none) -> Connector_JST:JST_XH_B6B-XH-A_1x06_P2.50mm_Vertical
- J206: value (none) -> JST_Couleur_3V; footprint (none) -> Connector_JST:JST_XH_B4B-XH-A_1x04_P2.50mm_Vertical
- J207: value (none) -> JST_Couleur_1B; footprint (none) -> Connector_JST:JST_XH_B3B-XH-A_1x03_P2.50mm_Vertical
- R301, R302: value (none) -> 10k
- R303, R304: value (none) -> NC
Changed lines of the file:
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@@
       (effects (font (size 1.27 1.27)) (justify left))
     )
-    (property "Value" "" (id 1) (at 40.64 123.19 0)
+    (property "Value" "10k" (id 1) (at 40.64 123.19 0)
       (effects (font (size 1.27 1.27)) (justify left))
     )
@@
       (effects (font (size 1.27 1.27)) (justify left))
     )
-    (property "Value" "" (id 1) (at 110.49 55.8799 0)
-      (effects (font (size 1.27 1.27)) (justify left))
-    )
-    (property "Footprint" "" (id 2) (at 107.95 54.61 0)
+    (property "Value" "JST_Bordure_2" (id 1) (at 110.49 55.8799 0)
+      (effects (font (size 1.27 1.27)) (justify left))
+    )
+    (property "Footprint" "Connector_JST:JST_XH_B3B-XH-A_1x03_P2.50mm_Vertical" (id 2) (at 107.95 54.61 0)
       (effects (font (size 1.27 1.27)) hide)
     )
@@
       (effects (font (size 1.27 1.27)) hide)
     )
-    (property "Value" "" (id 1) (at 95.25 54.61 90))
+    (property "Value" "+5V" (id 1) (at 95.25 54.61 90))
     (property "Footprint" "" (id 2) (at 100.33 54.61 0)
       (effects (font (size 1.27 1.27)) hide)
@@
       (effects (font (size 1.27 1.27)) (justify left))
     )
-    (property "Value" "" (id 1) (at 255.27 57.1499 0)
-      (effects (font (size 1.27 1.27)) (justify left))
-    )
-    (property "Footprint" "" (id 2) (at 252.73 55.88 0)
+    (property "Value" "JST_Couleur_1B" (id 1) (at 255.27 57.1499 0)
+      (effects (font (size 1.27 1.27)) (justify left))
+    )
+    (property "Footprint" "Connector_JST:JST_XH_B3B-XH-A_1x03_P2.50mm_Vertical" (id 2) (at 252.73 55.88 0)
       (effects (font (size 1.27 1.27)) hide)
     )
@@
       (effects (font (size 1.27 1.27)) (justify left))
     )
-    (property "Value" "" (id 1) (at 59.69 55.8799 0)
-      (effects (font (size 1.27 1.27)) (justify left))
-    )
-    (property "Footprint" "" (id 2) (at 57.15 54.61 0)
+    (property "Value" "JST_Bordure_1" (id 1) (at 59.69 55.8799 0)
+      (effects (font (size 1.27 1.27)) (justify left))
+    )
+    (property "Footprint" "Connector_JST:JST_XH_B3B-XH-A_1x03_P2.50mm_Vertical" (id 2) (at 57.15 54.61 0)
       (effects (font (size 1.27 1.27)) hide)
     )
@@
       (effects (font (size 1.27 1.27)) (justify left))
     )
-    (property "Value" "" (id 1) (at 228.6 128.2699 0)
-      (effects (font (size 1.27 1.27)) (justify left))
-    )
-    (property "Footprint" "" (id 2) (at 226.06 125.73 0)
+    (property "Value" "JST_Couleur_3V" (id 1) (at 228.6 128.2699 0)
+      (effects (font (size 1.27 1.27)) (justify left))
+    )
+    (property "Footprint" "Connector_JST:JST_XH_B4B-XH-A_1x04_P2.50mm_Vertical" (id 2) (at 226.06 125.73 0)
       (effects (font (size 1.27 1.27)) hide)
     )
@@
       (effects (font (size 1.27 1.27)) (justify left))
     )
-    (property "Value" "" (id 1) (at 105.41 123.19 0)
+    (property "Value" "NC" (id 1) (at 105.41 123.19 0)
       (effects (font (size 1.27 1.27)) (justify left))
     )
@@
       (effects (font (size 1.27 1.27)) hide)
     )
-    (property "Value" "" (id 1) (at 118.11 113.03 90))
+    (property "Value" "+5V" (id 1) (at 118.11 113.03 90))
     (property "Footprint" "" (id 2) (at 118.11 119.38 0)
       (effects (font (size 1.27 1.27)) hide)
@@
       (effects (font (size 1.27 1.27)) hide)
     )
-    (property "Value" "" (id 1) (at 93.98 52.07 90)
+    (property "Value" "GND" (id 1) (at 93.98 52.07 90)
       (effects (font (size 1.27 1.27)) (justify left))
     )
@@
       (effects (font (size 1.27 1.27)) (justify left))
     )
-    (property "Value" "" (id 1) (at 222.25 55.8799 0)
-      (effects (font (size 1.27 1.27)) (justify left))
-    )
-    (property "Footprint" "" (id 2) (at 219.71 53.34 0)
+    (property "Value" "JST_Couleur_1A" (id 1) (at 222.25 55.8799 0)
+      (effects (font (size 1.27 1.27)) (justify left))
+    )
+    (property "Footprint" "Connector_JST:JST_XH_B6B-XH-A_1x06_P2.50mm_Vertical" (id 2) (at 219.71 53.34 0)
       (effects (font (size 1.27 1.27)) hide)
     )
@@
       (effects (font (size 1.27 1.27)) hide)
     )
-    (property "Value" "" (id 1) (at 214.63 123.1899 90)
+    (property "Value" "GND" (id 1) (at 214.63 123.1899 90)
       (effects (font (size 1.27 1.27)) (justify right))
     )
@@
       (effects (font (size 1.27 1.27)) hide)
     )
-    (property "Value" "" (id 1) (at 50.8 124.46 0))
+    (property "Value" "GND" (id 1) (at 50.8 124.46 0))
     (property "Footprint" "" (id 2) (at 54.61 123.19 0)
       (effects (font (size 1.27 1.27)) hide)
@@
       (effects (font (size 1.27 1.27)) hide)
     )
-    (property "Value" "" (id 1) (at 208.28 50.7999 90)
+    (property "Value" "GND" (id 1) (at 208.28 50.7999 90)
       (effects (font (size 1.27 1.27)) (justify right))
     )
@@
       (effects (font (size 1.27 1.27)) hide)
     )
-    (property "Value" "" (id 1) (at 114.3 123.19 0))
+    (property "Value" "GND" (id 1) (at 114.3 123.19 0))
     (property "Footprint" "" (id 2) (at 116.84 123.19 0)
       (effects (font (size 1.27 1.27)) hide)
@@
       (effects (font (size 1.27 1.27)) hide)
     )
-    (property "Value" "" (id 1) (at 214.63 130.8099 90)
+    (property "Value" "+5V" (id 1) (at 214.63 130.8099 90)
       (effects (font (size 1.27 1.27)) (justify left))
     )
@@
       (effects (font (size 1.27 1.27)) (justify left))
     )
-    (property "Value" "" (id 1) (at 92.71 125.73 0)
+    (property "Value" "NC" (id 1) (at 92.71 125.73 0)
       (effects (font (size 1.27 1.27)) (justify left))
     )
@@
       (effects (font (size 1.27 1.27)) hide)
     )
-    (property "Value" "" (id 1) (at 46.99 54.6099 90)
+    (property "Value" "+5V" (id 1) (at 46.99 54.6099 90)
       (effects (font (size 1.27 1.27)) (justify left))
     )
@@
       (effects (font (size 1.27 1.27)) hide)
     )
-    (property "Value" "" (id 1) (at 43.18 52.07 90)
+    (property "Value" "GND" (id 1) (at 43.18 52.07 90)
       (effects (font (size 1.27 1.27)) (justify left))
     )
@@
       (effects (font (size 1.27 1.27)) hide)
     )
-    (property "Value" "" (id 1) (at 54.61 113.03 0))
+    (property "Value" "+5V" (id 1) (at 54.61 113.03 0))
     (property "Footprint" "" (id 2) (at 54.61 118.11 0)
       (effects (font (size 1.27 1.27)) hide)
@@
       (effects (font (size 1.27 1.27)) hide)
     )
-    (property "Value" "" (id 1) (at 208.28 48.2599 90)
+    (property "Value" "+5V" (id 1) (at 208.28 48.2599 90)
       (effects (font (size 1.27 1.27)) (justify left))
     )
@@
       (effects (font (size 1.27 1.27)) (justify left))
     )
-    (property "Value" "" (id 1) (at 29.21 125.73 0)
+    (property "Value" "10k" (id 1) (at 29.21 125.73 0)
       (effects (font (size 1.27 1.27)) (justify left))
     )
@@
       (effects (font (size 1.27 1.27)) (justify left))
     )
-    (property "Value" "" (id 1) (at 127 128.2699 0)
-      (effects (font (size 1.27 1.27)) (justify left))
-    )
-    (property "Footprint" "" (id 2) (at 124.46 125.73 0)
+    (property "Value" "JST_TOF_2" (id 1) (at 127 128.2699 0)
+      (effects (font (size 1.27 1.27)) (justify left))
+    )
+    (property "Footprint" "Connector_JST:JST_XH_B6B-XH-A_1x06_P2.50mm_Vertical" (id 2) (at 124.46 125.73 0)
       (effects (font (size 1.27 1.27)) hide)
     )
@@
       (effects (font (size 1.27 1.27)) (justify left))
     )
-    (property "Value" "" (id 1) (at 64.77 128.2699 0)
-      (effects (font (size 1.27 1.27)) (justify left))
-    )
-    (property "Footprint" "" (id 2) (at 62.23 125.73 0)
-      (effects (font (size 1.27 1.27)) hide)
-    )
+    (property "Value" "JST_TOF_1" (id 1) (at 64.77 128.2699 0)
+      (effects (font (size 1.27 1.27)) (justify left))
+    )
+    (property "Footprint" "Connector_JST:JST_XH_B6B-XH-A_1x06_P2.50mm_Vertical" (id 2) (at 62.23 125.73 0)
+      (effects (font (size 1.27 1.27)) hide)
+    )
