File: Hardware/KiCad_Schematic_PCB_v2/Actionneurs.kicad_sch (KiCad schematic)
At the start: 22 parts, among them J502 JST_driver1, J503 JST_driver2, J504 JST_servomoteur, U503 ZXBM5210-S, U504 ZXBM5210-S

Commit message: Final placement
Connections:
- net TIM_Driver1_CH1: now also JP503.2 (B), U503.4 (FWD)
- net TIM_Driver1_CH1N: now also JP504.2 (B), U503.5 (REV)
- net TIM_Driver2_CH1: now also JP508.2 (B), U504.4 (FWD)
- net TIM_Driver2_CH1N: now also JP509.2 (B), U504.5 (REV)
- net TIM_Encoder1_CH1: now also J502.3 (Pin_3), JP501.2 (B)
- net TIM_Encoder1_CH2: now also J502.4 (Pin_4), JP502.2 (B)
- net TIM_Encoder2_CH1: now also J503.3 (Pin_3), JP506.2 (B)
- net TIM_Encoder2_CH2: now also J503.4 (Pin_4), JP507.2 (B)
- net +7.2_U504: now reaches C507.1, C508.1, JP510.2 (B), U504.2 (VM), U504.3 (VDD), U504.6 (VREF)
- net +7.2_U504: now also C505.1, C506.1, JP505.2 (B), U503.2 (VM), U503.3 (VDD), U503.6 (VREF)
Other:
- moved on the sheet: JP501, JP502, JP506, JP507, JP508, JP509
