File: Hardware/KiCad_Schematic_PCB_v2/Projet_robot_ESE.kicad_pcb (KiCad board)
At the start: 4 copper layers, 110 x 50 mm, 66 parts, among them J201 JST_Bordure_1, J202 JST_TOF_1, J203 JST_TOF_2, J204 JST_Bordure_2, J205 JST_Couleur_1A, J206 JST_Couleur_3V, J207 JST_Couleur_1B, J208 Conn_02x07_Odd_Even, J209 JST_SUPP, J501 JST_switch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

Commit message: Final placement
Parts:
- J209: footprint Connector_JST:JST_XH_B6B-XH-A_1x06_P2.50mm_Vertical -> Connector_PinHeader_2.54mm:PinHeader_1x06_P2.54mm_Vertical
- moved D501 26.7 mm to (97.4, 49.2), turned to 180 degrees
- moved R501 22.9 mm to (94.9, 50.5), turned to -90 degrees
- moved D202 20.1 mm to (112.2, 42.0)
- moved D201 20.1 mm to (112.2, 44.1)
- moved R202 20.1 mm to (116.7, 44.1)
- moved R203 20.1 mm to (116.6, 42.0)
- moved C504 17.2 mm to (100.2, 50.1), turned to -90 degrees
- moved C502 17.0 mm to (105.8, 61.0), turned to 0 degrees
- moved C503 16.6 mm to (109.0, 51.0), turned to 180 degrees
- moved U501 15.1 mm to (107.8, 67.0)
- moved U502 15.0 mm to (104.8, 50.0), turned to 180 degrees
- moved C501 14.6 mm to (109.7, 61.0), turned to 0 degrees
- moved JP202 12.0 mm to (47.9, 47.4), turned to 0 degrees
- moved J206 9.05 mm to (28.5, 45.0), turned to 90 degrees
- moved C205 5.53 mm to (89.2, 46.5)
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Connections:
- net Net-(C205-Pad1) renamed /STM32/OSC_IN
- net Net-(C206-Pad1) renamed /STM32/OSC_OUT
- net Net-(D501-Pad2) renamed /Alimentation/LED
- C504 pad 2: Net-(C504-Pad2) -> +3.3V
- C505 pad 1: Net-(C505-Pad1) -> /Actionneurs/+7.2_U504
- C506 pad 1: Net-(C505-Pad1) -> /Actionneurs/+7.2_U504
- C507 pad 1: Net-(C507-Pad1) -> /Actionneurs/+7.2_U504
- C508 pad 1: Net-(C507-Pad1) -> /Actionneurs/+7.2_U504
- J205 pad 3: /Capteurs/LED_CC -> /Capteurs/S2
- J205 pad 4: /Capteurs/S2 -> /Capteurs/S3
- J205 pad 5: /Capteurs/S3 -> /Capteurs/LED_CC
- J207 pad 1: /Capteurs/S0 -> /Capteurs/OE
- J207 pad 2: /Capteurs/S1 -> /Capteurs/S0
- J207 pad 3: /Capteurs/OE -> /Capteurs/S1
- J208 pad 13: Net-(J208-Pad13) -> UART_STLink_RX
- J208 pad 14: Net-(J208-Pad14) -> UART_STLink_TX
- J502 pad 3: Net-(J502-Pad3) -> /Actionneurs/TIM_Encoder1_CH1
- J502 pad 4: Net-(J502-Pad4) -> /Actionneurs/TIM_Encoder1_CH2
- J503 pad 3: Net-(J503-Pad3) -> /Actionneurs/TIM_Encoder2_CH1
- J503 pad 4: Net-(J503-Pad4) -> /Actionneurs/TIM_Encoder2_CH2
- JP201 pad 2: Net-(J208-Pad13) -> UART_STLink_RX
- JP202 pad 1: Net-(J208-Pad14) -> UART_STLink_TX
- JP501 pad 2: Net-(J502-Pad3) -> /Actionneurs/TIM_Encoder1_CH1
- JP502 pad 2: Net-(J502-Pad4) -> /Actionneurs/TIM_Encoder1_CH2
- JP503 pad 2: Net-(JP503-Pad2) -> /Actionneurs/TIM_Driver1_CH1
- JP504 pad 2: Net-(JP504-Pad2) -> /Actionneurs/TIM_Driver1_CH1N
- JP505 pad 2: Net-(C505-Pad1) -> /Actionneurs/+7.2_U504
- JP506 pad 2: Net-(J503-Pad3) -> /Actionneurs/TIM_Encoder2_CH1
- JP507 pad 2: Net-(J503-Pad4) -> /Actionneurs/TIM_Encoder2_CH2
- JP508 pad 2: Net-(JP508-Pad2) -> /Actionneurs/TIM_Driver2_CH1
- JP509 pad 2: Net-(JP509-Pad2) -> /Actionneurs/TIM_Driver2_CH1N
- JP510 pad 2: Net-(C507-Pad1) -> /Actionneurs/+7.2_U504
- U501 pad 1: GND -> +BATT
- U501 pad 2: +5V -> GND
- U501 pad 3: +BATT -> +5V
- U502 pad 5: Net-(C504-Pad2) -> +3.3V
- U503 pad 2: Net-(C505-Pad1) -> /Actionneurs/+7.2_U504
- U503 pad 3: Net-(C505-Pad1) -> /Actionneurs/+7.2_U504
- U503 pad 4: Net-(JP503-Pad2) -> /Actionneurs/TIM_Driver1_CH1
- U503 pad 5: Net-(JP504-Pad2) -> /Actionneurs/TIM_Driver1_CH1N
- U503 pad 6: Net-(C505-Pad1) -> /Actionneurs/+7.2_U504
- U504 pad 2: Net-(C507-Pad1) -> /Actionneurs/+7.2_U504
- U504 pad 3: Net-(C507-Pad1) -> /Actionneurs/+7.2_U504
- U504 pad 4: Net-(JP508-Pad2) -> /Actionneurs/TIM_Driver2_CH1
- U504 pad 5: Net-(JP509-Pad2) -> /Actionneurs/TIM_Driver2_CH1N
- U504 pad 6: Net-(C507-Pad1) -> /Actionneurs/+7.2_U504
Routing:
- net +3.3V: track 0.00 -> 1.55 mm, vias 0 -> 7
- net GND: track 0.00 -> 0.10 mm, vias 0 -> 28
- net +BATT: track 0.00 -> 0.08 mm, vias 0 -> 6
- net +5V: vias 0 -> 8
- added copper zone on In2.Cu, net +3.3V
- added copper zone on In2.Cu, net +BATT
- added copper zone on In1.Cu, net GND
- removed copper zone on In1.Cu, net (none)
