File: Hardware/KiCad_Schematic_PCB_v2/STM32.kicad_sch (KiCad schematic)
At the start: 17 parts, among them J208 Conn_02x07_Odd_Even, J209 JST_SUPP, U201 STM32G070RBT6, Y201 16MHz

Commit message: Final placement
Parts:
- J209: footprint Connector_JST:JST_XH_B6B-XH-A_1x06_P2.50mm_Vertical -> Connector_PinHeader_2.54mm:PinHeader_1x06_P2.54mm_Vertical
Connections:
- net UART_STLink_RX: now also J208.13 (Pin_13), JP201.2 (B)
- net UART_STLink_TX: now also J208.14 (Pin_14), JP202.1 (A)
- net OSC_OUT: now reaches C206.1, R201.2, Y201.1
- net OSC_IN: now reaches C205.1, U201.10 (PF0_OSC_IN), Y201.3
