File: Hardware/KiCad_Schematic_PCB_v2/capteurs_v2.kicad_sch (KiCad schematic)
At the start: 11 parts, among them J201 JST_Bordure_1, J202 JST_TOF_1, J203 JST_TOF_2, J204 JST_Bordure_2, J205 JST_Couleur_1A, J206 JST_Couleur_3V, J207 JST_Couleur_1B

Commit message: Final placement
Connections:
- net LED_CC: now also J205.5 (Pin_5); no longer J205.3 (Pin_3)
- net OE: now also J207.1 (Pin_1); no longer J207.3 (Pin_3)
- net S0: now also J207.2 (Pin_2); no longer J207.1 (Pin_1)
- net S1: now also J207.3 (Pin_3); no longer J207.2 (Pin_2)
- net S2: now also J205.3 (Pin_3); no longer J205.4 (Pin_4)
- net S3: now also J205.4 (Pin_4); no longer J205.5 (Pin_5)
Changed lines of the file:
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@@
+    (stroke (width 0) (type default) (color 0 0 0 0))
+  )
+  (wire (pts (xy 213.36 55.88) (xy 214.63 55.88))
     (stroke (width 0) (type default) (color 0 0 0 0))
   )
@@
     (effects (font (size 1.27 1.27)) (justify right))
   )
-  (hierarchical_label "OE" (shape input) (at 247.65 58.42 180)
+  (hierarchical_label "OE" (shape input) (at 247.65 53.34 180)
     (effects (font (size 1.27 1.27)) (justify right))
   )
@@
     (effects (font (size 1.27 1.27)) (justify right))
   )
-  (hierarchical_label "S3" (shape input) (at 214.63 58.42 180)
+  (hierarchical_label "S3" (shape input) (at 213.36 55.88 180)
     (effects (font (size 1.27 1.27)) (justify right))
   )
@@
     (effects (font (size 1.27 1.27)) (justify right))
   )
-  (hierarchical_label "S1" (shape input) (at 247.65 55.88 180)
+  (hierarchical_label "S1" (shape input) (at 247.65 58.42 180)
     (effects (font (size 1.27 1.27)) (justify right))
   )
@@
     (effects (font (size 1.27 1.27)) (justify right))
   )
-  (hierarchical_label "LED_CC" (shape input) (at 213.36 53.34 180)
+  (hierarchical_label "LED_CC" (shape input) (at 214.63 58.42 180)
     (effects (font (size 1.27 1.27)) (justify right))
   )
@@
     (effects (font (size 1.27 1.27)) (justify right))
   )
-  (hierarchical_label "S2" (shape input) (at 214.63 55.88 180)
+  (hierarchical_label "S2" (shape input) (at 213.36 53.34 180)
     (effects (font (size 1.27 1.27)) (justify right))
   )
-  (hierarchical_label "S0" (shape input) (at 247.65 53.34 180)
+  (hierarchical_label "S0" (shape input) (at 247.65 55.88 180)
     (effects (font (size 1.27 1.27)) (justify right))
   )
