File: Hardware/Projet_robot_ESE/Actionneurs.kicad_sch (KiCad schematic)
At the start: 22 parts, among them J502 JST_driver1, J503 JST_driver2, J504 JST_servomoteur, U503 ZXBM5210-S, U504 ZXBM5210-S

Commit message: Update servomoteur
Parts:
- added R502: 10k, Resistor_SMD:R_0603_1608Metric_Pad0.98x0.95mm_HandSolder, symbol Device:R_Small
Connections:
- net UART_XL320: now also R502.2
- new net +3.3V: R502.1
Changed lines of the file:
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@@
   (junction (at 234.95 139.7) (diameter 0) (color 0 0 0 0)
   )
+  (junction (at 242.57 137.16) (diameter 0) (color 0 0 0 0)
+  )
   (junction (at 200.66 51.181) (diameter 0) (color 0 0 0 0)
   )
@@
     (stroke (width 0) (type default) (color 0 0 0 0))
   )
+  (wire (pts (xy 242.57 125.73) (xy 242.57 128.27))
+    (stroke (width 0) (type default) (color 0 0 0 0))
+  )
   (wire (pts (xy 200.66 53.467) (xy 202.057 53.467))
     (stroke (width 0) (type default) (color 0 0 0 0))
@@
     (stroke (width 0) (type default) (color 0 0 0 0))
   )
+  (wire (pts (xy 238.76 137.16) (xy 242.57 137.16))
+    (stroke (width 0) (type default) (color 0 0 0 0))
+  )
   (wire (pts (xy 214.63 59.563) (xy 217.17 59.563))
     (stroke (width 0) (type default) (color 0 0 0 0))
@@
     (stroke (width 0) (type default) (color 0 0 0 0))
   )
+  (wire (pts (xy 242.57 137.16) (xy 245.11 137.16))
+    (stroke (width 0) (type default) (color 0 0 0 0))
+  )
   (wire (pts (xy 75.057 71.374) (xy 75.057 52.578))
     (stroke (width 0) (type default) (color 0 0 0 0))
@@
   )
   (wire (pts (xy 121.92 166.37) (xy 121.92 160.02))
+    (stroke (width 0) (type default) (color 0 0 0 0))
+  )
+  (wire (pts (xy 242.57 133.35) (xy 242.57 137.16))
     (stroke (width 0) (type default) (color 0 0 0 0))
   )
@@
     (effects (font (size 1.27 1.27)) (justify right))
   )
-  (hierarchical_label "UART_XL320" (shape input) (at 245.11 137.16 180)
+  (hierarchical_label "UART_XL320" (shape input) (at 238.76 137.16 180)
     (effects (font (size 1.27 1.27)) (justify right))
   )
@@
     (pin "2")
   )
+  (symbol (lib_id "Device:R_Small") (at 242.57 130.81 0) (unit 1)
+    (in_bom yes) (on_board yes) (fields_autoplaced)
+    (property "Reference" "R502" (id 0) (at 245.11 129.5399 0)
+      (effects (font (size 1.27 1.27)) (justify left))
+    )
+    (property "Value" "10k" (id 1) (at 245.11 132.0799 0)
+      (effects (font (size 1.27 1.27)) (justify left))
+    )
+    (property "Footprint" "Resistor_SMD:R_0603_1608Metric_Pad0.98x0.95mm_HandSolder" (id 2) (at 242.57 130.81 0)
+      (effects (font (size 1.27 1.27)) hide)
+    )
+    (property "Datasheet" "~" (id 3) (at 242.57 130.81 0)
+      (effects (font (size 1.27 1.27)) hide)
+    )
+    (pin "1")
+    (pin "2")
+  )
   (symbol (lib_id "power:GND") (at 208.788 53.467 0) (unit 1)
     (in_bom yes) (on_board yes)
@@
   )
   (symbol (lib_id "Connector_Generic:Conn_01x03") (at 250.19 139.7 0) (mirror x) (unit 1)
-    (in_bom yes) (on_board yes) (fields_autoplaced)
-    (property "Reference" "J504" (id 0) (at 250.19 130.81 0))
-    (property "Value" "JST_servomoteur" (id 1) (at 250.19 133.35 0))
+    (in_bom yes) (on_board yes)
+    (property "Reference" "J504" (id 0) (at 262.89 137.16 0))
+    (property "Value" "JST_servomoteur" (id 1) (at 262.89 139.7 0))
     (property "Footprint" "Connector_JST:JST_XH_B3B-XH-A_1x03_P2.50mm_Vertical" (id 2) (at 250.19 139.7 0)
       (effects (font (size 1.27 1.27)) hide)
@@
       (effects (font (size 1.27 1.27)) hide)
     )
+    (pin "1")
+  )
+  (symbol (lib_id "power:+3.3V") (at 242.57 125.73 0) (unit 1)
+    (in_bom yes) (on_board yes) (fields_autoplaced)
+    (property "Reference" "#PWR0103" (id 0) (at 242.57 129.54 0)
+      (effects (font (size 1.27 1.27)) hide)
+    )
+    (property "Value" "+3.3V" (id 1) (at 242.57 120.65 0))
+    (property "Footprint" "" (id 2) (at 242.57 125.73 0)
+      (effects (font (size 1.27 1.27)) hide)
+    )
+    (property "Datasheet" "" (id 3) (at 242.57 125.73 0)
+      (effects (font (size 1.27 1.27)) hide)
+    )
