File: Hardware/Projet_robot_ESE/Projet_robot_ESE.kicad_pcb (KiCad board)
At the start: 4 copper layers, 110 x 50 mm, 67 parts, among them J201 JST_Bordure_1, J202 JST_TOF_1, J203 JST_TOF_2, J204 JST_Bordure_2, J205 JST_Couleur_1A, J206 JST_Couleur_3V, J207 JST_Couleur_1B, J208 Conn_02x07_Odd_Even, J209 JST_SUPP, J501 JST_switch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

Commit message: Update servomoteur
Parts:
- added R502: 10k, Resistor_SMD:R_0603_1608Metric_Pad0.98x0.95mm_HandSolder, F.Cu at (69.3, 66.5)
Routing:
- net +3.3V: track 14.7 -> 40.6 mm, vias 7 -> 8
- net /Actionneurs/UART_XL320: track 23.7 -> 24.9 mm
Changed lines of the file:
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@@
     (property "Sheetname" "Actionneurs")
     (attr through_hole)
-    (fp_text reference "J503" (at -5.18 -0.635) (layer "F.SilkS")
+    (fp_text reference "J503" (at -4.39 -0.025 90) (layer "F.SilkS")
       (effects (font (size 1 1) (thickness 0.15)))
     )
@@
     )
   )
+  (footprint "Resistor_SMD:R_0603_1608Metric_Pad0.98x0.95mm_HandSolder" (layer "F.Cu")
+    (at 69.29 66.54 180)
+    (descr "Resistor SMD 0603 (1608 Metric), square (rectangular) end terminal, IPC_7351 nominal with elongated pad for handsoldering. (Body size source: IPC-SM-782 page 72, https://www.pcb-3d.com/wordpress/wp-content/uploads/ipc-sm-782a_amendment_1_and_2.pdf), generated with kicad-footprint-generator")
+    (tags "resistor handsolder")
+    (property "Sheetfile" "Actionneurs.kicad_sch")
+    (property "Sheetname" "Actionneurs")
+    (attr smd)
+    (fp_text reference "R502" (at 0 1.5) (layer "F.SilkS")
+      (effects (font (size 1 1) (thickness 0.15)))
+    )
+    (fp_text value "10k" (at 0 1.43) (layer "F.Fab")
+      (effects (font (size 1 1) (thickness 0.15)))
+    )
+    (fp_text user "${REFERENCE}" (at 0 0) (layer "F.Fab")
+      (effects (font (size 0.4 0.4) (thickness 0.06)))
+    )
+    (fp_line (start -0.254724 -0.5225) (end 0.254724 -0.5225) (layer "F.SilkS") (width 0.12))
+    (fp_line (start -0.254724 0.5225) (end 0.254724 0.5225) (layer "F.SilkS") (width 0.12))
+    (fp_line (start -1.65 0.73) (end -1.65 -0.73) (layer "F.CrtYd") (width 0.05))
+    (fp_line (start 1.65 -0.73) (end 1.65 0.73) (layer "F.CrtYd") (width 0.05))
+    (fp_line (start -1.65 -0.73) (end 1.65 -0.73) (layer "F.CrtYd") (width 0.05))
+    (fp_line (start 1.65 0.73) (end -1.65 0.73) (layer "F.CrtYd") (width 0.05))
+    (fp_line (start 0.8 0.4125) (end -0.8 0.4125) (layer "F.Fab") (width 0.1))
+    (fp_line (start -0.8 0.4125) (end -0.8 -0.4125) (layer "F.Fab") (width 0.1))
+    (fp_line (start 0.8 -0.4125) (end 0.8 0.4125) (layer "F.Fab") (width 0.1))
+    (fp_line (start -0.8 -0.4125) (end 0.8 -0.4125) (layer "F.Fab") (width 0.1))
+    (pad "1" smd roundrect (at -0.9125 0 180) (size 0.975 0.95) (layers "F.Cu" "F.Paste" "F.Mask") (roundrect_rratio 0.25)
+      (net 1 "+3.3V") (pintype "passive"))
+    (pad "2" smd roundrect (at 0.9125 0 180) (size 0.975 0.95) (layers "F.Cu" "F.Paste" "F.Mask") (roundrect_rratio 0.25)
+      (net 49 "/Actionneurs/UART_XL320") (pintype "passive"))
+    (model "${KICAD6_3DMODEL_DIR}/Resistor_SMD.3dshapes/R_0603_1608Metric.wrl"
+      (offset (xyz 0 0 0))
+      (scale (xyz 1 1 1))
+      (rotate (xyz 0 0 0))
+    )
+  )
   (footprint "LED_SMD:LED_0603_1608Metric_Pad1.05x0.95mm_HandSolder" (layer "F.Cu")
     (at 97.51 47.74 180)
@@
     (property "Sheetname" "Actionneurs")
     (attr through_hole)
-    (fp_text reference "J502" (at 6.3 -4.385) (layer "F.SilkS")
+    (fp_text reference "J502" (at 17 0.375 90) (layer "F.SilkS")
       (effects (font (size 1 1) (thickness 0.15)))
     )
@@
     (property "Sheetname" "Actionneurs")
     (attr through_hole)
-    (fp_text reference "J504" (at 2.26 5.415) (layer "F.SilkS")
+    (fp_text reference "J504" (at 9.06 0.215 90) (layer "F.SilkS")
       (effects (font (size 1 1) (thickness 0.15)))
     )
@@
   (segment (start 100.25 50.49) (end 100.25 49.56) (width 0.75) (layer "F.Cu") (net 1))
   (segment (start 82.9275 46.03) (end 82.8175 46.14) (width 0.75) (layer "F.Cu") (net 1))
+  (segment (start 76.19 66.54) (end 76.69 66.04) (width 0.5) (layer "F.Cu") (net 1))
   (segment (start 84.245 47.88) (end 83.3675 47.88) (width 0.75) (layer "F.Cu") (net 1))
   (segment (start 103.72 49.54) (end 103.7425 49.5175) (width 0.75) (layer "F.Cu") (net 1))
@@
   (segment (start 84.225 46.03) (end 82.9275 46.03) (width 0.75) (layer "F.Cu") (net 1))
   (segment (start 94.99 49.9425) (end 94.97 49.9225) (width 0.75) (layer "F.Cu") (net 1))
+  (segment (start 70.2025 66.54) (end 76.19 66.54) (width 0.5) (layer "F.Cu") (net 1))
   (segment (start 94.99 50.8) (end 94.99 49.9425) (width 0.75) (layer "F.Cu") (net 1))
   (segment (start 80.705 45.94) (end 82.6175 45.94) (width 0.3) (layer "F.Cu") (net 1))
@@
   (via (at 57.99 43.22) (size 0.8) (drill 0.4) (layers "F.Cu" "B.Cu") (free) (net 1))
   (via (at 83.3075 47.94) (size 0.8) (drill 0.4) (layers "F.Cu" "B.Cu") (free) (net 1))
+  (via (at 76.69 66.04) (size 0.8) (drill 0.4) (layers "F.Cu" "B.Cu") (net 1))
   (via (at 82.8175 46.14) (size 0.8) (drill 0.4) (layers "F.Cu" "B.Cu") (net 1))
   (via (at 100.25 50.49) (size 0.8) (drill 0.4) (layers "F.Cu" "B.Cu") (free) (net 1))
   (via (at 94.99 50.8) (size 0.8) (drill 0.4) (layers "F.Cu" "B.Cu") (free) (net 1))
+  (segment (start 76.69 66.04) (end 76.69 58.44) (width 0.5) (layer "B.Cu") (net 1))
+  (segment (start 76.69 58.44) (end 83.3475 51.7825) (width 0.5) (layer "B.Cu") (net 1))
+  (segment (start 83.3475 51.7825) (end 83.3475 49.66) (width 0.5) (layer "B.Cu") (net 1))
   (segment (start 98.385 47.74) (end 98.385 46.445) (width 0.75) (layer "F.Cu") (net 2))
   (segment (start 107.257122 47.949281) (end 106.638903 48.5675) (width 0.5) (layer "F.Cu") (net 2))
@@
   (segment (start 81.73 70.885) (end 81.2 71.415) (width 0.5) (layer "F.Cu") (net 48))
   (segment (start 81.73 65.277918) (end 81.73 70.885) (width 0.5) (layer "F.Cu") (net 48))
+  (segment (start 67.335 65.985) (end 66.65 66.67) (width 0.3) (layer "F.Cu") (net 49))
+  (segment (start 67.89 66.54) (end 67.335 65.985) (width 0.3) (layer "F.Cu") (net 49))
   (segment (start 74.28 50.865) (end 74.28 59.04) (width 0.3) (layer "F.Cu") (net 49))
   (segment (start 66.65 66.67) (end 66.65 71.355) (width 0.3) (layer "F.Cu") (net 49))
-  (segment (start 74.28 59.04) (end 66.65 66.67) (width 0.3) (layer "F.Cu") (net 49))
+  (segment (start 68.3775 66.54) (end 67.89 66.54) (width 0.3) (layer "F.Cu") (net 49))
+  (segment (start 74.28 59.04) (end 67.335 65.985) (width 0.3) (layer "F.Cu") (net 49))
   (segment (start 61.53 37.12) (end 61.46 37.12) (width 0.3) (layer "F.Cu") (net 50))
   (segment (start 60.55 38.03) (end 60.065 38.03) (width 0.3) (layer "F.Cu") (net 50))
