File: Hardware/Capteur_couleur/Capteur_couleur.kicad_pcb (KiCad board)
At the start: 2 copper layers, 32 x 21.5 mm, 18 parts, among them J101 JST_Couleur_3V, U101 VEML3328, U102 MCP1802x-xx02xOT

Commit message: Update Capteur couleur
Other:
- board text added: "Alix HAVRET Loïcia KOEHL Quentin SIMON Chelsea COMLAN"
- board text added: "Capteur couleur VEML3328"
Changed lines of the file:
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@@
   (gr_arc (start 131 62.5) (mid 129.681981 65.681981) (end 126.5 67) (layer "Edge.Cuts") (width 0.1))
   (gr_line (start 103 67) (end 126.5 67) (layer "Edge.Cuts") (width 0.1))
+  (gr_text "Alix HAVRET\nLoïcia KOEHL\nQuentin SIMON\nChelsea COMLAN" (at 126.6 58.8) (layer "F.SilkS")
+    (effects (font (size 0.4 0.4) (thickness 0.1)))
+  )
+  (gr_text "Capteur couleur \nVEML3328" (at 126.5 55) (layer "F.SilkS")
+    (effects (font (size 0.5 0.5) (thickness 0.1)))
+  )
   (segment (start 107.6 54) (end 105 54) (width 0.75) (layer "F.Cu") (net 1))
   (segment (start 101 58.5) (end 101 60) (width 0.75) (layer "F.Cu") (net 1))

Commit message: Update footprint
Parts:
- moved R102 0.10 mm to (117.7, 58.6)
Routing:
- net SCL: track 19.6 -> 19.1 mm
Changed lines of the file:
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@@
     (property "Sheetname" "")
     (attr smd)
-    (fp_text reference "U101" (at -0.1 -1.1 unlocked) (layer "F.SilkS")
+    (fp_text reference "U101" (at 0 -1.1 unlocked) (layer "F.SilkS")
       (effects (font (size 0.5 0.5) (thickness 0.1)))
     )
@@
       (effects (font (size 1 1) (thickness 0.15)))
     )
-    (fp_rect (start -0.99 -0.59) (end 1.01 0.66) (layer "F.SilkS") (width 0.01) (fill none))
-    (pad "1" smd roundrect (at -0.7525 -0.315) (size 0.425 0.35) (layers "F.Cu" "F.Paste" "F.Mask") (roundrect_rratio 0.25)
+    (fp_line (start -1 -0.59) (end 1 -0.59) (layer "F.SilkS") (width 0.12))
+    (fp_line (start -1 -0.05) (end -1 0.1) (layer "F.SilkS") (width 0.12))
+    (fp_line (start 1 -0.05) (end 1 0.1) (layer "F.SilkS") (width 0.12))
+    (fp_line (start -1 0.66) (end 1 0.66) (layer "F.SilkS") (width 0.12))
+    (pad "1" smd roundrect (at -0.95 -0.315) (size 0.9 0.35) (layers "F.Cu" "F.Paste" "F.Mask") (roundrect_rratio 0.25)
       (net 2 "GND") (pinfunction "GND") (pintype "power_in"))
-    (pad "2" smd roundrect (at -0.7525 0.385) (size 0.425 0.35) (layers "F.Cu" "F.Paste" "F.Mask") (roundrect_rratio 0.25)
+    (pad "2" smd roundrect (at -0.95 0.385) (size 0.9 0.35) (layers "F.Cu" "F.Paste" "F.Mask") (roundrect_rratio 0.25)
       (net 8 "SDA") (pinfunction "SDA") (pintype "bidirectional"))
-    (pad "3" smd roundrect (at 0.7225 0.385) (size 0.525 0.35) (layers "F.Cu" "F.Paste" "F.Mask") (roundrect_rratio 0.25)
+    (pad "3" smd roundrect (at 0.9 0.385) (size 1 0.35) (layers "F.Cu" "F.Paste" "F.Mask") (roundrect_rratio 0.25)
       (net 9 "SCL") (pinfunction "SCL") (pintype "bidirectional"))
-    (pad "4" smd roundrect (at 0.785 -0.315) (size 0.4 0.35) (layers "F.Cu" "F.Paste" "F.Mask") (roundrect_rratio 0.25)
+    (pad "4" smd roundrect (at 0.95 -0.315) (size 0.9 0.35) (layers "F.Cu" "F.Paste" "F.Mask") (roundrect_rratio 0.25)
       (net 3 "+3.3V") (pinfunction "VDD") (pintype "power_in"))
   )
@@
     (property "Sheetname" "")
     (attr smd)
-    (fp_text reference "U102" (at 0 -2.4) (layer "F.SilkS")
+    (fp_text reference "U102" (at 0 2.3) (layer "F.SilkS")
       (effects (font (size 0.5 0.5) (thickness 0.1)))
     )
@@
     (property "Sheetname" "")
     (attr smd)
-    (fp_text reference "C103" (at -0.0525 1.285) (layer "F.SilkS")
+    (fp_text reference "C103" (at 0.8475 1.185) (layer "F.SilkS")
       (effects (font (size 0.5 0.5) (thickness 0.1)))
     )
@@
   )
   (footprint "Resistor_SMD:R_0603_1608Metric_Pad0.98x0.95mm_HandSolder" (layer "F.Cu")
-    (at 117.6 58.6 -90)
+    (at 117.7 58.6 -90)
     (descr "Resistor SMD 0603 (1608 Metric), square (rectangular) end terminal, IPC_7351 nominal with elongated pad for handsoldering. (Body size source: IPC-SM-782 page 72, https://www.pcb-3d.com/wordpress/wp-content/uploads/ipc-sm-782a_amendment_1_and_2.pdf), generated with kicad-footprint-generator")
     (tags "resistor handsolder")
@@
   (segment (start 102.3625 58.25) (end 102.4625 58.35) (width 0.25) (layer "F.Cu") (net 1))
   (segment (start 102.3625 55.9) (end 102.3625 58.25) (width 0.75) (layer "F.Cu") (net 1))
-  (segment (start 115.035 57.785) (end 115.2475 57.9975) (width 0.5) (layer "F.Cu") (net 2))
-  (segment (start 114.5475 57.785) (end 115.035 57.785) (width 0.5) (layer "F.Cu") (net 2))
+  (segment (start 115.2 58.266282) (end 115.2 59.3) (width 0.3) (layer "F.Cu") (net 2))
+  (segment (start 114.718718 57.785) (end 115.2 58.266282) (width 0.3) (layer "F.Cu") (net 2))
+  (segment (start 114.35 57.785) (end 114.718718 57.785) (width 0.3) (layer "F.Cu") (net 2))
   (segment (start 115.2475 59.2525) (end 115.15 59.35) (width 0.5) (layer "F.Cu") (net 2))
-  (segment (start 115.2475 57.9975) (end 115.2475 59.2525) (width 0.5) (layer "F.Cu") (net 2))
+  (segment (start 115.2 59.3) (end 115.15 59.35) (width 0.3) (layer "F.Cu") (net 2))
   (via (at 115.15 59.35) (size 0.8) (drill 0.4) (layers "F.Cu" "B.Cu") (free) (net 2))
   (via (at 109.3 54.6) (size 0.8) (drill 0.4) (layers "F.Cu" "B.Cu") (free) (net 2))
@@
   (segment (start 115.92 56.9) (end 116.21 56.61) (width 0.75) (layer "F.Cu") (net 3))
   (segment (start 105.83125 58.23125) (end 105.7125 58.35) (width 0.25) (layer "F.Cu") (net 3))
+  (segment (start 116.25 57.23) (end 115.92 56.9) (width 0.3) (layer "F.Cu") (net 3))
   (segment (start 107.0875 56.975) (end 106.8 57.2625) (width 0.75) (layer "F.Cu") (net 3))
   (segment (start 110.75 57.775) (end 110.7 57.825) (width 0.25) (layer "F.Cu") (net 3))
@@
   (segment (start 105.7125 58.35) (end 104.7375 58.35) (width 0.75) (layer "F.Cu") (net 3))
   (segment (start 108.8 63.425) (end 107.225 63.425) (width 0.75) (layer "F.Cu") (net 3))
+  (segment (start 116.25 57.785) (end 117.5025 57.785) (width 0.3) (layer "F.Cu") (net 3))
   (segment (start 106.8 57.2625) (end 105.83125 58.23125) (width 0.75) (layer "F.Cu") (net 3))
-  (segment (start 117.6 57.6875) (end 116.1825 57.6875) (width 0.5) (layer "F.Cu") (net 3))
   (segment (start 123.3 56) (end 124.1 56.8) (width 0.75) (layer "F.Cu") (net 3))
   (segment (start 116.21 55.585) (end 116.21 56.61) (width 0.75) (layer "F.Cu") (net 3))
+  (segment (start 117.5025 57.785) (end 117.6 57.6875) (width 0.3) (layer "F.Cu") (net 3))
   (segment (start 106.2 62.4) (end 106.2 58.6) (width 0.75) (layer "F.Cu") (net 3))
+  (segment (start 116.25 57.785) (end 116.25 57.23) (width 0.3) (layer "F.Cu") (net 3))
   (segment (start 122.575 63.525) (end 120.1 63.525) (width 0.75) (layer "F.Cu") (net 3))
-  (segment (start 116.21 56.61) (end 116.21 57.66) (width 0.5) (layer "F.Cu") (net 3))
   (segment (start 107.225 63.425) (end 106.2 62.4) (width 0.75) (layer "F.Cu") (net 3))
   (segment (start 109 59.6125) (end 110.6625 59.6125) (width 0.5) (layer "F.Cu") (net 4))
@@
   (segment (start 121.875 59.4625) (end 121.9125 59.5) (width 0.25) (layer "F.Cu") (net 7))
   (segment (start 113.25 49.475) (end 113.25 49.75) (width 0.25) (layer "F.Cu") (net 8))
-  (segment (start 112.9 59.6) (end 113.4325 59.6) (width 0.5) (layer "F.Cu") (net 8))
-  (segment (start 113.4325 59.6) (end 114.5475 58.485) (width 0.5) (layer "F.Cu") (net 8))
+  (segment (start 114.015 58.485) (end 112.9 59.6) (width 0.3) (layer "F.Cu") (net 8))
   (segment (start 112.75 50.25) (end 112.75 53.45) (width 0.5) (layer "F.Cu") (net 8))
   (segment (start 112.9 61.3) (end 112.9 59.6) (width 0.5) (layer "F.Cu") (net 8))
   (segment (start 112.75 53.45) (end 112 54.2) (width 0.5) (layer "F.Cu") (net 8))
+  (segment (start 114.35 58.485) (end 114.015 58.485) (width 0.3) (layer "F.Cu") (net 8))
   (segment (start 113.25 49.75) (end 112.75 50.25) (width 0.5) (layer "F.Cu") (net 8))
   (via (at 112.9 61.3) (size 0.8) (drill 0.4) (layers "F.Cu" "B.Cu") (net 8))
@@
   (segment (start 112.9 61.3) (end 112 60.4) (width 0.5) (layer "B.Cu") (net 8))
   (segment (start 115.75 49.75) (end 115.25 50.25) (width 0.5) (layer "F.Cu") (net 9))
-  (segment (start 116.4125 59.5125) (end 116.0225 59.1225) (width 0.5) (layer "F.Cu") (net 9))
+  (segment (start 116.5725 58.485) (end 117.6 59.5125) (width 0.3) (layer "F.Cu") (net 9))
   (segment (start 117.6 61.5) (end 117.6 59.5125) (width 0.5) (layer "F.Cu") (net 9))
-  (segment (start 116.0225 59.1225) (end 116.0225 58.5125) (width 0.5) (layer "F.Cu") (net 9))
   (segment (start 115.25 53.35) (end 115.9 54) (width 0.5) (layer "F.Cu") (net 9))
-  (segment (start 117.6 59.5125) (end 116.4125 59.5125) (width 0.5) (layer "F.Cu") (net 9))
+  (segment (start 116.2 58.485) (end 116.5725 58.485) (width 0.3) (layer "F.Cu") (net 9))
   (segment (start 115.75 49.475) (end 115.75 49.75) (width 0.25) (layer "F.Cu") (net 9))
   (segment (start 115.25 50.25) (end 115.25 53.35) (width 0.5) (layer "F.Cu") (net 9))
